Commit message: Added a new version of the ik_demo. The old one now is named ik_demo_wrist. The new one now opens the gripper first and then moves the tcp (new link and fixed joint defined in the xacro file) to the ball.

File: robot_description/urdf/robot.xacro (robot description, xacro)
@@ -184,4 +184,13 @@
   </collision>
 </link>
+<link name="tcp_link">
+  <visual>
+    <origin xyz="0 0 0" rpy="0 0 0"/>
+    <geometry>
+      <sphere radius="0.005"/>
+    </geometry>
+    <material name="blue"/>
+  </visual>
+</link>
 <joint name="joint1" type="revolute">
   <origin xyz="-0.01268 0.001996 0.10629" rpy="0 0 0"/>
@@ -243,3 +252,9 @@
   <mimic joint="joint_plate" multiplier="38.79"/>
 </joint>
+<joint name="tcp_fixed_joint" type="fixed">
+  <parent link="link4_1"/>
+  <child link="tcp_link"/>
+  <!-- Adjust the XYZ offset to place the TCP properly -->
+  <origin xyz="0.1 0 0" rpy="0 0 0"/>
+</joint>
 </robot>

Commit message: Made the tcp link invisible. Before it was visible as a ball

File: robot_description/urdf/robot.xacro (robot description, xacro)
@@ -187,8 +187,4 @@
   <visual>
     <origin xyz="0 0 0" rpy="0 0 0"/>
-    <geometry>
-      <sphere radius="0.005"/>
-    </geometry>
-    <material name="blue"/>
   </visual>
 </link>

Commit message: Moved the tcp to better represent the center point of the tool

File: robot_description/urdf/robot.xacro (robot description, xacro)
@@ -252,5 +252,5 @@
   <child link="tcp_link"/>
   <!-- Adjust the XYZ offset to place the TCP properly -->
-  <origin xyz="0.1 0 0" rpy="0 0 0"/>
+  <origin xyz="0.11 0 -0.01" rpy="0 0 0"/>
 </joint>
 </robot>

Commit message: Changed the Nullposition of the robot. For this reason, many things had to be updated: URDF, Limits, kinematic

File: robot_description/urdf/robot.xacro (robot description, xacro)
@@ -6,12 +6,12 @@
 <link name="base_link">
   <inertial>
-    <origin xyz="-0.0679401062157721 0.0014277216725000752 0.0384137562968467" rpy="0 0 0"/>
-    <mass value="3.1478109"/>
-    <inertia ixx="0.052924" iyy="0.098855" izz="0.120214" ixy="0.000123" iyz="-0.00015" ixz="0.001855"/>
+    <origin xyz="-0.01525516398344423 0.011844787362381164 0.03066554293773624" rpy="0 0 0"/>
+    <mass value="13.800576305987779"/>
+    <inertia ixx="0.052926" iyy="0.098856" izz="0.120212" ixy="7.3e-05" iyz="-0.000151" ixz="0.001895"/>
   </inertial>
   <visual>
     <origin xyz="0 0 0" rpy="0 0 0"/>
     <geometry>
-      <mesh filename="file://$(find robot_description)/meshes/base_link.stl" scale="0.001 0.001 0.001"/>
+      <mesh filename="package://robot_description/meshes/base_link.stl" scale="0.001 0.001 0.001"/>
     </geometry>
     <material name="silver"/>
@@ -20,5 +20,65 @@
     <origin xyz="0 0 0" rpy="0 0 0"/>
     <geometry>
-      <mesh filename="file://$(find robot_description)/meshes/base_link.stl" scale="0.001 0.001 0.001"/>
+      <mesh filename="package://robot_description/meshes/base_link.stl" scale="0.001 0.001 0.001"/>
+    </geometry>
+  </collision>
+</link>
+<link name="finger1_1">
+  <inertial>
+    <origin xyz="0.017766259815813923 0.019470567148479057 -0.0003130477037422419" rpy="0 0 0"/>
+    <mass value="0.007627104997040501"/>
+    <inertia ixx="1e-06" iyy="4e-06" izz="5e-06" ixy="-1e-06" iyz="-0.0" ixz="-0.0"/>
+  </inertial>
+  <visual>
+    <origin xyz="-0.649164 0.031879 -0.130769" rpy="0 0 0"/>
+    <geometry>
+      <mesh filename="package://robot_description/meshes/finger1_1.stl" scale="0.001 0.001 0.001"/>
+    </geometry>
+    <material name="silver"/>
+  </visual>
+  <collision>
+    <origin xyz="-0.649164 0.031879 -0.130769" rpy="0 0 0"/>
+    <geometry>
+      <mesh filename="package://robot_description/meshes/finger1_1.stl" scale="0.001 0.001 0.001"/>
+    </geometry>
+  </collision>
+</link>
+<link name="finger3_1">
+  <inertial>
+    <origin xyz="0.016557095492733764 -0.009289304587601917 0.01651813436684768" rpy="0 0 0"/>
+    <mass value="0.008118325054343886"/>
+    <inertia ixx="1e-06" iyy="5e-06" izz="5e-06" ixy="1e-06" iyz="0.0" ixz="-1e-06"/>
+  </inertial>
+  <visual>
+    <origin xyz="-0.649071 -0.035625 -0.091805" rpy="0 0 0"/>
+    <geometry>
+      <mesh filename="package://robot_description/meshes/finger3_1.stl" scale="0.001 0.001 0.001"/>
+    </geometry>
+    <material name="silver"/>
+  </visual>
+  <collision>
+    <origin xyz="-0.649071 -0.035625 -0.091805" rpy="0 0 0"/>
+    <geometry>
+      <mesh filename="package://robot_description/meshes/finger3_1.stl" scale="0.001 0.001 0.001"/>
+    </geometry>
+  </collision>
+</link>
+<link name="finger2_1">
+  <inertial>
+    <origin xyz="0.016435817583313028 -0.009686132400900348 -0.016410363628854535" rpy="0 0 0"/>
+    <mass value="0.008118323730919927"/>
+    <inertia ixx="1e-06" iyy="5e-06" izz="5e-06" ixy="1e-06" iyz="-0.0" ixz="1e-06"/>
+  </inertial>
+  <visual>
+    <origin xyz="-0.64911 -0.035617 -0.169747" rpy="0 0 0"/>
+    <geometry>
+      <mesh filename="package://robot_description/meshes/finger2_1.stl" scale="0.001 0.001 0.001"/>
+    </geometry>
+    <material name="silver"/>
+  </visual>
+  <collision>
+    <origin xyz="-0.64911 -0.035617 -0.169747" rpy="0 0 0"/>
+    <geometry>
+      <mesh filename="package://robot_description/meshes/finger2_1.stl" scale="0.001 0.001 0.001"/>
     </geometry>
   </collision>
@@ -26,19 +86,19 @@
 <link name="link1_1">
   <inertial>
-    <origin xyz="0.009853212349380608 -0.0013058822796042395 0.03681261950807038" rpy="0 0 0"/>
-    <mass value="2.6592794"/>
-    <inertia ixx="0.011723" iyy="0.040532" izz="0.039189" ixy="-0.00052" iyz="7.7e-05" ixz="0.002459"/>
-  </inertial>
-  <visual>
-    <origin xyz="0.01268 -0.001996 -0.10629" rpy="0 0 0"/>
-    <geometry>
-      <mesh filename="file://$(find robot_description)/meshes/link1_1.stl" scale="0.001 0.001 0.001"/>
-    </geometry>
-    <material name="silver"/>
-  </visual>
-  <collision>
-    <origin xyz="0.01268 -0.001996 -0.10629" rpy="0 0 0"/>
-    <geometry>
-      <mesh filename="file://$(find robot_description)/meshes/link1_1.stl" scale="0.001 0.001 0.001"/>
+    <origin xyz="0.009870752041433603 -0.0012985996197881471 0.0283066433531641" rpy="0 0 0"/>
+    <mass value="7.642342288589914"/>
+    <inertia ixx="0.011727" iyy="0.04053" izz="0.039186" ixy="-0.000551" iyz="8e-05" ixz="0.002475"/>
+  </inertial>
+  <visual>
+    <origin xyz="-0.04005 -0.012465 -0.106459" rpy="0 0 0"/>
+    <geometry>
+      <mesh filename="package://robot_description/meshes/link1_1.stl" scale="0.001 0.001 0.001"/>
+    </geometry>
+    <material name="silver"/>
+  </visual>
+  <collision>
+    <origin xyz="-0.04005 -0.012465 -0.106459" rpy="0 0 0"/>
+    <geometry>
+      <mesh filename="package://robot_description/meshes/link1_1.stl" scale="0.001 0.001 0.001"/>
     </geometry>
   </collision>
@@ -46,19 +106,19 @@
 <link name="link2_1">
   <inertial>
-    <origin xyz="0.07785203265870212 0.006684318764593031 0.06532544373999474" rpy="0 0 0"/>
-    <mass value="0.94268266"/>
-    <inertia ixx="0.015526" iyy="0.026356" izz="0.019554" ixy="0.002104" iyz="0.001765" ixz="-0.011421"/>
-  </inertial>
-  <visual>
-    <origin xyz="-0.09387 -0.001996 -0.15129" rpy="0 0 0"/>
-    <geometry>
-      <mesh filename="file://$(find robot_description)/meshes/link2_1.stl" scale="0.001 0.001 0.001"/>
-    </geometry>
-    <material name="silver"/>
-  </visual>
-  <collision>
-    <origin xyz="-0.09387 -0.001996 -0.15129" rpy="0 0 0"/>
-    <geometry>
-      <mesh filename="file://$(find robot_description)/meshes/link2_1.stl" scale="0.001 0.001 0.001"/>
+    <origin xyz="0.10159804902516775 0.02779415868097769 -5.765765416601565e-05" rpy="0 0 0"/>
+    <mass value="4.531072242141342"/>
+    <inertia ixx="0.005937" iyy="0.026362" izz="0.029137" ixy="0.002724" iyz="-2e-06" ixz="1.4e-05"/>
+  </inertial>
+  <visual>
+    <origin xyz="-0.146644 0.008424 -0.142894" rpy="0 0 0"/>
+    <geometry>
+      <mesh filename="package://robot_description/meshes/link2_1.stl" scale="0.001 0.001 0.001"/>
+    </geometry>
+    <material name="silver"/>
+  </visual>
+  <collision>
+    <origin xyz="-0.146644 0.008424 -0.142894" rpy="0 0 0"/>
+    <geometry>
+      <mesh filename="package://robot_description/meshes/link2_1.stl" scale="0.001 0.001 0.001"/>
     </geometry>
   </collision>
@@ -66,19 +126,19 @@
 <link name="link3_1">
   <inertial>
-    <origin xyz="0.08865319906030028 0.008333660765872107 0.03226660259352443" rpy="0 0 0"/>
-    <mass value="0.53015345"/>
-    <inertia ixx="0.003579" iyy="0.012679" izz="0.012845" ixy="0.001413" iyz="0.000514" ixz="-0.003887"/>
-  </inertial>
-  <visual>
-    <origin xyz="-0.2624 -0.001996 -0.292704" rpy="0 0 0"/>
-    <geometry>
-      <mesh filename="file://$(find robot_description)/meshes/link3_1.stl" scale="0.001 0.001 0.001"/>
-    </geometry>
-    <material name="silver"/>
-  </visual>
-  <collision>
-    <origin xyz="-0.2624 -0.001996 -0.292704" rpy="0 0 0"/>
-    <geometry>
-      <mesh filename="file://$(find robot_description)/meshes/link3_1.stl" scale="0.001 0.001 0.001"/>
+    <origin xyz="0.09430665017480633 0.033435499071081135 -4.474360302914038e-05" rpy="0 0 0"/>
+    <mass value="1.942633915240748"/>
+    <inertia ixx="0.002161" iyy="0.012682" izz="0.01426" ixy="0.001492" iyz="-1e-06" ixz="6e-06"/>
+  </inertial>
+  <visual>
+    <origin xyz="-0.366648 0.012186 -0.142763" rpy="0 0 0"/>
+    <geometry>
+      <mesh filename="package://robot_description/meshes/link3_1.stl" scale="0.001 0.001 0.001"/>
+    </geometry>
+    <material name="silver"/>
+  </visual>
+  <collision>
+    <origin xyz="-0.366648 0.012186 -0.142763" rpy="0 0 0"/>
+    <geometry>
+      <mesh filename="package://robot_description/meshes/link3_1.stl" scale="0.001 0.001 0.001"/>
     </geometry>
   </collision>
@@ -86,19 +146,19 @@
 <link name="link4_1">
   <inertial>
-    <origin xyz="0.03760750782340139 0.007481639102787173 -0.007913875947465843" rpy="0 0 0"/>
-    <mass value="0.119"/>
-    <inertia ixx="0.000355" iyy="0.000164" izz="0.00024" ixy="-8e-06" iyz="1e-06" ixz="3e-06"/>
-  </inertial>
-  <visual>
-    <origin xyz="-0.469133 -0.001996 -0.367948" rpy="0 0 0"/>
-    <geometry>
-      <mesh filename="file://$(find robot_description)/meshes/link4_1.stl" scale="0.001 0.001 0.001"/>
-    </geometry>
-    <material name="silver"/>
-  </visual>
-  <collision>
-    <origin xyz="-0.469133 -0.001996 -0.367948" rpy="0 0 0"/>
-    <geometry>
-      <mesh filename="file://$(find robot_description)/meshes/link4_1.stl" scale="0.001 0.001 0.001"/>
+    <origin xyz="0.040594015010658735 0.007526480171399416 -0.011433358935294402" rpy="0 0 0"/>
+    <mass value="0.2862169162828504"/>
+    <inertia ixx="0.000355" iyy="0.000164" izz="0.00024" ixy="-7e-06" iyz="1e-06" ixz="3e-06"/>
+  </inertial>
+  <visual>
+    <origin xyz="-0.586621 -0.013052 -0.142653" rpy="0 0 0"/>
+    <geometry>
+      <mesh filename="package://robot_description/meshes/link4_1.stl" scale="0.001 0.001 0.001"/>
+    </geometry>
+    <material name="silver"/>
+  </visual>
+  <collision>
+    <origin xyz="-0.586621 -0.013052 -0.142653" rpy="0 0 0"/>
+    <geometry>
+      <mesh filename="package://robot_description/meshes/link4_1.stl" scale="0.001 0.001 0.001"/>
     </geometry>
   </collision>
@@ -106,79 +166,19 @@
 <link name="plate_1">
   <inertial>
-    <origin xyz="-0.5152768789930368 0.359593601257941 -0.0019849464337260425" rpy="0 0 0"/>
+    <origin xyz="0.002936460578468969 -3.32136638021667e-06 1.0551585629070548e-05" rpy="0 0 0"/>
     <mass value="0.005591792200815245"/>
     <inertia ixx="1e-06" iyy="1e-06" izz="1e-06" ixy="0.0" iyz="0.0" ixz="-0.0"/>
   </inertial>
   <visual>
-    <origin xyz="-1.03536 0.357604 -0.361597" rpy="0 0 0"/>
-    <geometry>
-      <mesh filename="file://$(find robot_description)/meshes/plate_1.stl" scale="0.001 0.001 0.001"/>
-    </geometry>
-    <material name="silver"/>
-  </visual>
-  <collision>
-    <origin xyz="-1.03536 0.357604 -0.361597" rpy="0 0 0"/>
-    <geometry>
-      <mesh filename="file://$(find robot_description)/meshes/plate_1.stl" scale="0.001 0.001 0.001"/>
-    </geometry>
-  </collision>
-</link>
-<link name="finger1_1">
-  <inertial>
-    <origin xyz="0.017787445914003053 0.01945172295891951 -0.00030579074354203373" rpy="0 0 0"/>
-    <mass value="0.007627104997040501"/>
-    <inertia ixx="1e-06" iyy="4e-06" izz="5e-06" ixy="-1e-06" iyz="-0.0" ixz="-0.0"/>
-  </inertial>
-  <visual>
-    <origin xyz="-0.528633 0.043004 -0.3596" rpy="0 0 0"/>
-    <geometry>
-      <mesh filename="file://$(find robot_description)/meshes/finger1_1.stl" scale="0.001 0.001 0.001"/>
-    </geometry>
-    <material name="silver"/>
-  </visual>
-  <collision>
-    <origin xyz="-0.528633 0.043004 -0.3596" rpy="0 0 0"/>
-    <geometry>
-      <mesh filename="file://$(find robot_description)/meshes/finger1_1.stl" scale="0.001 0.001 0.001"/>
-    </geometry>
-  </collision>
-</link>
-<link name="finger3_1">
-  <inertial>
-    <origin xyz="0.016538444380158834 -0.009305155777922368 0.01652756515622833" rpy="0 0 0"/>
-    <mass value="0.008118325054343886"/>
-    <inertia ixx="1e-06" iyy="5e-06" izz="5e-06" ixy="1e-06" iyz="0.0" ixz="-1e-06"/>
-  </inertial>
-  <visual>
-    <origin xyz="-0.528633 -0.024496 -0.320629" rpy="0 0 0"/>
-    <geometry>
-      <mesh filename="file://$(find robot_description)/meshes/finger3_1.stl" scale="0.001 0.001 0.001"/>
-    </geometry>
-    <material name="silver"/>
-  </visual>
-  <collision>
-    <origin xyz="-0.528633 -0.024496 -0.320629" rpy="0 0 0"/>
-    <geometry>
-      <mesh filename="file://$(find robot_description)/meshes/finger3_1.stl" scale="0.001 0.001 0.001"/>
-    </geometry>
-  </collision>
-</link>
-<link name="finger2_1">
-  <inertial>
-    <origin xyz="0.016432808719543224 -0.009705029513755988 -0.016400937312406938" rpy="0 0 0"/>
-    <mass value="0.008118323730919927"/>
-    <inertia ixx="1e-06" iyy="5e-06" izz="5e-06" ixy="1e-06" iyz="-0.0" ixz="1e-06"/>
-  </inertial>
-  <visual>
-    <origin xyz="-0.528633 -0.024496 -0.398571" rpy="0 0 0"/>
-    <geometry>
-      <mesh filename="file://$(find robot_description)/meshes/finger2_1.stl" scale="0.001 0.001 0.001"/>
-    </geometry>
-    <material name="silver"/>
-  </visual>
-  <collision>
-    <origin xyz="-0.528633 -0.024496 -0.398571" rpy="0 0 0"/>
-    <geometry>
-      <mesh filename="file://$(find robot_description)/meshes/finger2_1.stl" scale="0.001 0.001 0.001"/>
+    <origin xyz="-0.636482 -0.013107 -0.13078" rpy="0 0 0"/>
+    <geometry>
+      <mesh filename="package://robot_description/meshes/plate_1.stl" scale="0.001 0.001 0.001"/>
+    </geometry>
+    <material name="silver"/>
+  </visual>
+  <collision>
+    <origin xyz="-0.636482 -0.013107 -0.13078" rpy="0 0 0"/>
+    <geometry>
+      <mesh filename="package://robot_description/meshes/plate_1.stl" scale="0.001 0.001 0.001"/>
     </geometry>
   </collision>
@@ -186,65 +186,68 @@
 <link name="tcp_link">
   <visual>
-    <origin xyz="0 0 0" rpy="0 0 0"/>
-  </visual>
-</link>
+    <geometry>
+      <box size="0.01 0.01 0.01"/> <!-- or a mesh -->
+    </geometry>
+    <material name="blue"/>
+  </visual>
+</link>
+<joint name="joint_finger1" type="continuous">
+  <origin xyz="0.062543 -0.044931 -0.011884" rpy="0 0 0"/>
+  <parent link="link4_1"/>
+  <child link="finger1_1"/>
+  <axis xyz="-0.000509 0.000108 -1.0"/>
+  <mimic joint="joint_plate" multiplier="38.79"/>
+  <limit upper="0.349066" lower="0.0" effort="100.0" velocity="100"/>
+</joint>
+<joint name="joint_finger2" type="continuous">
+  <origin xyz="0.06245 0.022573 -0.050848" rpy="0 0 0"/>
+  <parent link="link4_1"/>
+  <child link="finger3_1"/>
+  <axis xyz="-0.000682 0.865971 0.500094"/>
+  <mimic joint="joint_plate" multiplier="38.79"/>
+  <limit upper="0.349066" lower="0.0" effort="100.0" velocity="100"/>
+</joint>
+<joint name="joint_finger3" type="continuous">
+  <origin xyz="0.062489 0.022565 0.027094" rpy="0 0 0"/>
+  <parent link="link4_1"/>
+  <child link="finger2_1"/>
+  <axis xyz="0.001191 -0.866079 0.499906"/>
+  <mimic joint="joint_plate" multiplier="38.79"/>
+  <limit upper="0.349066" lower="0.0" effort="100.0" velocity="100"/>
+</joint>
 <joint name="joint1" type="revolute">
-  <origin xyz="-0.01268 0.001996 0.10629" rpy="0 0 0"/>
+  <origin xyz="0.04005 0.012465 0.106459" rpy="0 0 0"/>
   <parent link="base_link"/>
   <child link="link1_1"/>
-  <axis xyz="-0.0 0.0 -1.0"/>
-  <limit upper="2.705593" lower="-2.5571593" effort="100.0" velocity="100"/>
+  <axis xyz="0.000594 -0.000107 1.0"/>
+  <limit upper="2.617994" lower="-2.617994" effort="100" velocity="100"/>
 </joint>
 <joint name="joint2" type="revolute">
-  <origin xyz="0.10655 0.0 0.045" rpy="0 0 0"/>
+  <origin xyz="0.106594 -0.020889 0.036435" rpy="0 0 0"/>
   <parent link="link1_1"/>
   <child link="link2_1"/>
-  <axis xyz="0.0 -1.0 0.0"/>
-  <limit upper="0.905796" lower="-1.016198" effort="100.0" velocity="100"/>
+  <axis xyz="0.001081 -0.999999 -0.000108"/>
+  <limit upper="1.658063" lower="0.0" effort="100" velocity="100"/>
 </joint>
 <joint name="joint3" type="revolute">
-  <origin xyz="0.16853 0.0 0.141414" rpy="0 0 0"/>
+  <origin xyz="0.220004 -0.003762 -0.000131" rpy="0 0 0"/>
   <parent link="link2_1"/>
   <child link="link3_1"/>
-  <axis xyz="0.0 -1.0 0.0"/>
-  <limit upper="2.330162" lower="-1.628862" effort="100.0" velocity="100"/>
+  <axis xyz="0.001081 -0.999999 -0.000108"/>
+  <limit upper="2.094395" lower="-2.007129" effort="100" velocity="100"/>
 </joint>
 <joint name="joint4" type="revolute">
-  <origin xyz="0.206733 0.0 0.075244" rpy="0 0 0"/>
+  <origin xyz="0.219973 0.025238 -0.00011" rpy="0 0 0"/>
   <parent link="link3_1"/>
   <child link="link4_1"/>
-  <axis xyz="-0.0 1.0 -0.0"/>
-  <limit upper="1.311329" lower="-2.087129" effort="100.0" velocity="100"/>
+  <axis xyz="-0.001081 0.999999 0.000108"/>
+  <limit upper="1.745329" lower="-1.570796" effort="100" velocity="100"/>
 </joint>
 <joint name="joint_plate" type="prismatic">
-  <origin xyz="0.566227 -0.3596 -0.006351" rpy="0 0 0"/>
+  <origin xyz="0.049861 5.5e-05 -0.011873" rpy="0 0 0"/>
   <parent link="link4_1"/>
   <child link="plate_1"/>
-  <axis xyz="1.0 0.0 0.0"/>
-  <limit upper="0.009" lower="0.0" effort="100.0" velocity="100"/>
-</joint>
-<joint name="joint_finger1" type="revolute">
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